Commit message: Update URDF to be used with Gazebo simulation

File: robots/edo_sim.urdf (robot description, URDF)
Before this commit: robot edo_sim, 7 links, 6 joints
Links:
- added link ee_link; collision box size=0.01 0.01 0.01
- added link tool0
- added link world
- link base_link: geometry collision mesh filename=package://edo_description/meshes/base_link.STL; visual mesh filename=package://edo_description/meshes/base_link.STL
- link link_1: geometry collision mesh filename=package://edo_description/meshes/link_1.STL; visual mesh filename=package://edo_description/meshes/link_1.STL
- link link_2: geometry collision mesh filename=package://edo_description/meshes/link_2.STL; visual mesh filename=package://edo_description/meshes/link_2.STL
- link link_3: geometry collision mesh filename=package://edo_description/meshes/link_3.STL; visual mesh filename=package://edo_description/meshes/link_3.STL
- link link_4: geometry collision mesh filename=package://edo_description/meshes/link_4.STL; visual mesh filename=package://edo_description/meshes/link_4.STL
- link link_5: geometry collision mesh filename=package://edo_description/meshes/link_5.STL; visual mesh filename=package://edo_description/meshes/link_5.STL
- link link_6: geometry collision mesh filename=package://edo_description/meshes/link_6.STL; visual mesh filename=package://edo_description/meshes/link_6.STL
Joints:
- added joint ee_fixed_joint: type fixed, parent link_6, child ee_link, origin xyz=0.0 0.0823 0.0 rpy=0.0 0.0 1.57079632679
- added joint link_6-tool0_fixed_joint: type fixed, parent link_6, child tool0, origin xyz=0 0.0823 0 rpy=-1.57079632679 0 0
- added joint world_joint: type fixed, parent world, child base_link, origin xyz=0.0 0.0 0.0 rpy=0.0 0.0 0.0
- joint joint_1: limit (none) -> lower=-6.28318530718 upper=6.28318530718 effort=150.0 velocity=3.15
- joint joint_2: limit (none) -> lower=-6.28318530718 upper=6.28318530718 effort=150.0 velocity=3.15
- joint joint_3: limit (none) -> lower=-6.28318530718 upper=6.28318530718 effort=150.0 velocity=3.15
- joint joint_4: limit (none) -> lower=-6.28318530718 upper=6.28318530718 effort=150.0 velocity=3.15
- joint joint_5: limit (none) -> lower=-6.28318530718 upper=6.28318530718 effort=150.0 velocity=3.15
- joint joint_6: limit (none) -> lower=-6.28318530718 upper=6.28318530718 effort=150.0 velocity=3.15
