Commit message: Update model files and correctly align links to match real world model

File: urdf/edo.urdf.xacro (robot description, xacro)
@@ -5,5 +5,5 @@
     <!--Import the lbr iiwa macro -->
     <xacro:include filename="$(find edo_description)/urdf/edo.xacro"/>
-    <xacro:arg name="hardware_interface" default="PositionJointInterface"/>
+    <xacro:arg name="hardware_interface" default="hardware_interface/PositionJointInterface"/>
     <xacro:arg name="robot_name" default="edo"/>
     <xacro:arg name="origin_xyz" default="0 0 0"/>

File: urdf/edo.xacro (robot description, xacro)
@@ -35,5 +35,5 @@
                 <origin xyz="0 0 0" rpy="0 0 0"/>
                 <geometry>
-                    <mesh filename="package://edo_description/meshes/base_link.STL"/>
+                    <mesh filename="package://edo_description/meshes/base_link.stl"/>
                 </geometry>
                 <material name="Grey"/>
@@ -42,5 +42,38 @@
                 <origin xyz="0 0 0" rpy="0 0 0"/>
                 <geometry>
-                    <mesh filename="package://edo_description/meshes/base_link.STL"/>
+                    <mesh filename="package://edo_description/meshes/base_link.stl"/>
+                </geometry>
+                <material name="Grey"/>
+            </collision>
+        </link>
+        <!-- joint between base_link and base_spacer -->
+        <joint name="${robot_name}_joint_spacer" type="fixed">
+            <parent link="${robot_name}_base_link"/>
+            <child link="${robot_name}_base_spacer_link"/>
+            <origin xyz="0 0 0.135" rpy="0 0 0"/>
+        </joint>
+        <link name="${robot_name}_base_spacer_link">
+            <inertial>
+                <origin xyz="0 0 0.005" rpy="0 0 0"/>
+                <mass value="0.01"/>
+                <inertia
+                        ixx="0.0123841200738068"
+                        ixy="-0.000187984913202787"
+                        ixz="-1.32683892634308E-06"
+                        iyy="7.0169034503364E-05"
+                        iyz="-9.17416945099319E-05"
+                        izz="0.0123862261905614" />
+            </inertial>
+            <visual>
+                <origin xyz="0 0 0" rpy="0 0 0"/>
+                <geometry>
+                    <mesh filename="package://edo_description/meshes/base_spacer.stl"/>
+                </geometry>
+                <material name="Grey"/>
+            </visual>
+            <collision>
+                <origin xyz="0 0 0" rpy="0 0 0"/>
+                <geometry>
+                    <mesh filename="package://edo_description/meshes/base_spacer.stl"/>
                 </geometry>
                 <material name="Grey"/>
@@ -51,6 +84,6 @@
             <parent link="${robot_name}_base_link"/>
             <child link="${robot_name}_link_1"/>
-            <origin xyz="0.057188 0.0059831 0.135" rpy="${PI/2} 0 -${PI}"/>
-            <axis xyz="0 1 0"/>
+            <origin xyz="0 0 ${0.135 + 0.202}" rpy="0 0 0"/>
+            <axis xyz="0 0 1"/>
             <limit lower="${-180 * PI / 180}" upper="${180 * PI / 180}"
                    effort="${max_effort}" velocity="${max_velocity}" />
@@ -70,14 +103,14 @@
             </inertial>
             <visual>
-                <origin xyz="0 0.015 0" rpy="0 0 0"/>
-                <geometry>
-                    <mesh filename="package://edo_description/meshes/link_1.STL"/>
-                </geometry>
-                <material name="Orange"/>
-            </visual>
-            <collision>
-                <origin xyz="0 0.015 0" rpy="0 0 0"/>
-                <geometry>
-                    <mesh filename="package://edo_description/meshes/link_1.STL"/>
+                <origin xyz="0 0 0" rpy="0 0 0"/>
+                <geometry>
+                    <mesh filename="package://edo_description/meshes/link_1.stl"/>
+                </geometry>
+                <material name="Orange"/>
+            </visual>
+            <collision>
+                <origin xyz="0 0 0" rpy="0 0 0"/>
+                <geometry>
+                    <mesh filename="package://edo_description/meshes/link_1.stl"/>
                 </geometry>
                 <material name="Orange"/>
@@ -87,6 +120,6 @@
             <parent link="${robot_name}_link_1"/>
             <child link="${robot_name}_link_2"/>
-            <origin xyz="0 0.202 0" rpy="0.94237 -0.4634 -0.11653"/>
-            <axis xyz="-0.88847 0.2908 0.35504"/>
+            <origin xyz="0 0 0" rpy="${PI /2} 0 0"/>
+            <axis xyz="0 0 1"/>
             <limit lower="${-113 * PI / 180}" upper="${113 * PI / 180}"
                    effort="${max_effort}" velocity="${max_velocity}" />
@@ -108,12 +141,12 @@
                 <origin xyz="0 0 0" rpy="0 0 0"/>
                 <geometry>
-                    <mesh filename="package://edo_description/meshes/link_2.STL"/>
-                </geometry>
-                <material name="Orange"/>
-            </visual>
-            <collision>
-                <origin xyz="0 0 0" rpy="0 0 0"/>
-                <geometry>
-                    <mesh filename="package://edo_description/meshes/link_2.STL"/>
+                    <mesh filename="package://edo_description/meshes/link_2.stl"/>
+                </geometry>
+                <material name="Orange"/>
+            </visual>
+            <collision>
+                <origin xyz="0 0 0" rpy="0 0 0"/>
+                <geometry>
+                    <mesh filename="package://edo_description/meshes/link_2.stl"/>
                 </geometry>
                 <material name="Orange"/>
@@ -123,6 +156,6 @@
             <parent link="${robot_name}_link_2"/>
             <child link="${robot_name}_link_3"/>
-            <origin xyz="-0.024558 0.12737 -0.16578" rpy="0.97336 -0.36296 2.8253"/>
-            <axis xyz="1 0 0"/>
+            <origin xyz="0 0.2105 0" rpy="0 ${PI} ${PI}"/>
+            <axis xyz="0 0 -1"/>
             <limit lower="${-113 * PI / 180}" upper="${113 * PI / 180}"
                    effort="${max_effort}" velocity="${max_velocity}" />
@@ -144,12 +177,12 @@
                 <origin xyz="0 0 0" rpy="0 0 0"/>
                 <geometry>
-                    <mesh filename="package://edo_description/meshes/link_3.STL"/>
-                </geometry>
-                <material name="Orange"/>
-            </visual>
-            <collision>
-                <origin xyz="0 0 0" rpy="0 0 0"/>
-                <geometry>
-                    <mesh filename="package://edo_description/meshes/link_3.STL"/>
+                    <mesh filename="package://edo_description/meshes/link_3.stl"/>
+                </geometry>
+                <material name="Orange"/>
+            </visual>
+            <collision>
+                <origin xyz="0 0 0" rpy="0 0 0"/>
+                <geometry>
+                    <mesh filename="package://edo_description/meshes/link_3.stl"/>
                 </geometry>
                 <material name="Orange"/>
@@ -159,6 +192,6 @@
             <parent link="${robot_name}_link_3"/>
             <child link="${robot_name}_link_4"/>
-            <origin xyz="0.0088 -0.158 0" rpy="-${PI / 2} 0 0"/>
-            <axis xyz="0 0 -1"/>
+            <origin xyz="0 -0.268 0" rpy="${PI / 2} 0 0"/>
+            <axis xyz="0 0 1"/>
             <limit lower="${-180 * PI / 180}" upper="${180 * PI / 180}"
                    effort="${max_effort}" velocity="${max_velocity}" />
@@ -178,14 +211,14 @@
             </inertial>
             <visual>
-                <origin xyz="0 0 -0.0053" rpy="0 0 0"/>
-                <geometry>
-                    <mesh filename="package://edo_description/meshes/link_4.STL"/>
-                </geometry>
-                <material name="Orange"/>
-            </visual>
-            <collision>
-                <origin xyz="0 0 -0.0053" rpy="0 0 0"/>
-                <geometry>
-                    <mesh filename="package://edo_description/meshes/link_4.STL"/>
+                <origin xyz="0 0 0" rpy="0 0 0"/>
+                <geometry>
+                    <mesh filename="package://edo_description/meshes/link_4.stl"/>
+                </geometry>
+                <material name="Orange"/>
+            </visual>
+            <collision>
+                <origin xyz="0 0 0" rpy="0 0 0"/>
+                <geometry>
+                    <mesh filename="package://edo_description/meshes/link_4.stl"/>
                 </geometry>
                 <material name="Orange"/>
@@ -195,6 +228,6 @@
             <parent link="${robot_name}_link_4"/>
             <child link="${robot_name}_link_5"/>
-            <origin xyz="0 0 -0.1105" rpy="${PI} 0 ${PI}"/>
-            <axis xyz="0 0 1"/>
+            <origin xyz="0 0 0" rpy="0 0 0"/>
+            <axis xyz="0 -1 0"/>
             <limit lower="${-104 * PI / 180}" upper="${104 * PI / 180}"
                    effort="${max_effort}" velocity="${max_velocity}" />
@@ -216,12 +249,12 @@
                 <origin xyz="0 0 0" rpy="0 0 0"/>
                 <geometry>
-                    <mesh filename="package://edo_description/meshes/link_5.STL"/>
-                </geometry>
-                <material name="Orange"/>
-            </visual>
-            <collision>
-                <origin xyz="0 0 0" rpy="0 0 0"/>
-                <geometry>
-                    <mesh filename="package://edo_description/meshes/link_5.STL"/>
+                    <mesh filename="package://edo_description/meshes/link_5.stl"/>
+                </geometry>
+                <material name="Orange"/>
+            </visual>
+            <collision>
+                <origin xyz="0 0 0" rpy="0 0 0"/>
+                <geometry>
+                    <mesh filename="package://edo_description/meshes/link_5.stl"/>
                 </geometry>
                 <material name="Orange"/>
@@ -231,6 +264,6 @@
             <parent link="${robot_name}_link_5"/>
             <child link="${robot_name}_link_6"/>
-            <origin xyz="-0.0039 0 0.168" rpy="-${PI / 2} 0 0"/>
-            <axis xyz="0 -1 0"/>
+            <origin xyz="0 0 0.1745" rpy="${PI} 0 0"/>
+            <axis xyz="0 0 -1"/>
             <limit lower="${-2700 * PI / 180}" upper="${2700 * PI / 180}"
                    effort="${max_effort}" velocity="${max_velocity}" />
@@ -254,14 +287,14 @@
             </inertial>
             <visual>
-                <origin xyz="0 0.0075 0" rpy="0 0 0"/>
-                <geometry>
-                    <mesh filename="package://edo_description/meshes/link_6.STL"/>
-                </geometry>
-                <material name="Orange"/>
-            </visual>
-            <collision>
-                <origin xyz="0 0.0075 0" rpy="0 0 0"/>
-                <geometry>
-                    <mesh filename="package://edo_description/meshes/link_6.STL"/>
+                <origin xyz="0 0 0" rpy="0 0 0"/>
+                <geometry>
+                    <mesh filename="package://edo_description/meshes/link_6.stl"/>
+                </geometry>
+                <material name="Orange"/>
+            </visual>
+            <collision>
+                <origin xyz="0 0 0" rpy="0 0 0"/>
+                <geometry>
+                    <mesh filename="package://edo_description/meshes/link_6.stl"/>
                 </geometry>
                 <material name="Orange"/>
@@ -271,13 +304,7 @@
             <parent link="${robot_name}_link_6"/>
             <child link="${robot_name}_link_ee"/>
-            <origin xyz="0.0 -0.0075 0" rpy="${PI/2} 0 0"/>
+            <origin xyz="0 0 0" rpy="0 0 0"/>
         </joint>
         <link name="${robot_name}_link_ee">
-            <collision>
-                <geometry>
-                    <box size="0.01 0.01 0.01"/>
-                </geometry>
-                <origin  xyz="0 0 0" rpy="0 0 0"/>
-            </collision>
         </link>
         <!--Extensions -->

Commit message: Update robot rotation to align all coordinate systems along world frame

File: urdf/edo.urdf.xacro (robot description, xacro)
@@ -8,5 +8,5 @@
     <xacro:arg name="robot_name" default="edo"/>
     <xacro:arg name="origin_xyz" default="0 0 0"/>
-    <xacro:arg name="origin_rpy" default="0 0 -1.57079632679"/>
+    <xacro:arg name="origin_rpy" default="0 0 0"/>
     <!-- Fix to world just for testing -->
     <link name="world"/>

File: urdf/edo.xacro (robot description, xacro)
@@ -49,5 +49,5 @@
             <parent link="${robot_name}_base_link"/>
             <child link="${robot_name}_base_spacer_link"/>
-            <origin xyz="0 0 0.135" rpy="0 0 ${PI / 2}"/>
+            <origin xyz="0 0 0.135" rpy="0 0 0"/>
         </joint>
         <link name="${robot_name}_base_spacer_link">
@@ -82,5 +82,5 @@
             <parent link="${robot_name}_base_link"/>
             <child link="${robot_name}_link_1"/>
-            <origin xyz="0 0 ${0.135 + 0.202}" rpy="0 0 ${PI / 2}"/>
+            <origin xyz="0 0 ${0.135 + 0.202}" rpy="0 0 0"/>
             <axis xyz="0 0 1"/>
             <limit lower="${-180 * PI / 180}" upper="${180 * PI / 180}"
@@ -262,6 +262,6 @@
             <parent link="${robot_name}_link_5"/>
             <child link="${robot_name}_link_6"/>
-            <origin xyz="0 0 0.1745" rpy="${PI} 0 0"/>
-            <axis xyz="0 0 -1"/>
+            <origin xyz="0 0 0.1745" rpy="0 0 0"/>
+            <axis xyz="0 0 1"/>
             <!-- MoveIt has problems with these huge limits -->
             <!--limit lower="${-2700 * PI / 180}" upper="${2700 * PI / 180}"
@@ -301,5 +301,5 @@
             <parent link="${robot_name}_link_6"/>
             <child link="${robot_name}_link_ee"/>
-            <origin xyz="0 0 0" rpy="${PI} 0 0"/>
+            <origin xyz="0 0 0" rpy="0 0 0"/>
         </joint>
         <link name="${robot_name}_link_ee">
