Commit message: Remove unused safety controller

File: urdf/edo.xacro (robot description, xacro)
@@ -8,6 +8,4 @@
     <xacro:include filename="$(find edo_description)/urdf/utilities.xacro" />
     <!-- some constants -->
-    <xacro:property name="safety_controller_k_pos" value="100" />
-    <xacro:property name="safety_controller_k_vel" value="2" />
     <xacro:property name="joint_damping" value="0.5" />
     <xacro:property name="max_effort" value="300"/>
@@ -268,8 +266,4 @@
             <limit lower="${-2700 * PI / 180}" upper="${2700 * PI / 180}"
                    effort="${max_effort}" velocity="${max_velocity}" />
-            <safety_controller soft_lower_limit="${-118 * PI / 180}"
-                               soft_upper_limit="${118 * PI / 180}"
-                               k_position="${safety_controller_k_pos}"
-                               k_velocity="${safety_controller_k_vel}"/>
             <dynamics damping="${joint_damping}"/>
         </joint>

Commit message: Set more realisitc max_velocity

File: urdf/edo.xacro (robot description, xacro)
@@ -10,5 +10,5 @@
     <xacro:property name="joint_damping" value="0.5" />
     <xacro:property name="max_effort" value="300"/>
-    <xacro:property name="max_velocity" value="10"/>
+    <xacro:property name="max_velocity" value="1.5"/>
     <xacro:macro name="edo" params="parent hardware_interface robot_name *origin">
         <!--joint between {parent} and base_link-->
@@ -264,5 +264,8 @@
             <origin xyz="0 0 0.1745" rpy="${PI} 0 0"/>
             <axis xyz="0 0 -1"/>
-            <limit lower="${-2700 * PI / 180}" upper="${2700 * PI / 180}"
+            <!-- MoveIt has problems with these huge limits -->
+            <!--limit lower="${-2700 * PI / 180}" upper="${2700 * PI / 180}"
+                   effort="${max_effort}" velocity="${max_velocity}" /-->
+            <limit lower="${-270 * PI / 180}" upper="${270 * PI / 180}"
                    effort="${max_effort}" velocity="${max_velocity}" />
             <dynamics damping="${joint_damping}"/>

Commit message: Rotate robot to match technical sheet drawing

File: urdf/edo.xacro (robot description, xacro)
@@ -49,5 +49,5 @@
             <parent link="${robot_name}_base_link"/>
             <child link="${robot_name}_base_spacer_link"/>
-            <origin xyz="0 0 0.135" rpy="0 0 0"/>
+            <origin xyz="0 0 0.135" rpy="0 0 ${PI / 2}"/>
         </joint>
         <link name="${robot_name}_base_spacer_link">
@@ -82,5 +82,5 @@
             <parent link="${robot_name}_base_link"/>
             <child link="${robot_name}_link_1"/>
-            <origin xyz="0 0 ${0.135 + 0.202}" rpy="0 0 0"/>
+            <origin xyz="0 0 ${0.135 + 0.202}" rpy="0 0 ${PI / 2}"/>
             <axis xyz="0 0 1"/>
             <limit lower="${-180 * PI / 180}" upper="${180 * PI / 180}"

Commit message: Correct rotation of axis 2,3 and 5

File: urdf/edo.xacro (robot description, xacro)
@@ -119,5 +119,5 @@
             <child link="${robot_name}_link_2"/>
             <origin xyz="0 0 0" rpy="${PI /2} 0 0"/>
-            <axis xyz="0 0 1"/>
+            <axis xyz="0 0 -1"/>
             <limit lower="${-113 * PI / 180}" upper="${113 * PI / 180}"
                    effort="${max_effort}" velocity="${max_velocity}" />
@@ -155,5 +155,5 @@
             <child link="${robot_name}_link_3"/>
             <origin xyz="0 0.2105 0" rpy="0 ${PI} ${PI}"/>
-            <axis xyz="0 0 -1"/>
+            <axis xyz="0 0 1"/>
             <limit lower="${-113 * PI / 180}" upper="${113 * PI / 180}"
                    effort="${max_effort}" velocity="${max_velocity}" />
@@ -227,5 +227,5 @@
             <child link="${robot_name}_link_5"/>
             <origin xyz="0 0 0" rpy="0 0 0"/>
-            <axis xyz="0 -1 0"/>
+            <axis xyz="0 1 0"/>
             <limit lower="${-104 * PI / 180}" upper="${104 * PI / 180}"
                    effort="${max_effort}" velocity="${max_velocity}" />

Commit message: Correctly orientate gripper and include griper ee in moveit

File: urdf/edo.xacro (robot description, xacro)
@@ -301,5 +301,5 @@
             <parent link="${robot_name}_link_6"/>
             <child link="${robot_name}_link_ee"/>
-            <origin xyz="0 0 0" rpy="0 0 0"/>
+            <origin xyz="0 0 0" rpy="${PI} 0 0"/>
         </joint>
         <link name="${robot_name}_link_ee">

Commit message: Add simplified collision models

File: urdf/edo.xacro (robot description, xacro)
@@ -33,5 +33,5 @@
                 <origin xyz="0 0 0" rpy="0 0 0"/>
                 <geometry>
-                    <mesh filename="package://edo_description/meshes/base_link.stl"/>
+                    <mesh filename="package://edo_description/meshes/visual/base_link.stl"/>
                 </geometry>
                 <material name="Grey"/>
@@ -40,5 +40,5 @@
                 <origin xyz="0 0 0" rpy="0 0 0"/>
                 <geometry>
-                    <mesh filename="package://edo_description/meshes/base_link.stl"/>
+                    <mesh filename="package://edo_description/meshes/collision/base_link.stl"/>
                 </geometry>
                 <material name="Grey"/>
@@ -66,5 +66,5 @@
                 <origin xyz="0 0 0" rpy="0 0 0"/>
                 <geometry>
-                    <mesh filename="package://edo_description/meshes/base_spacer.stl"/>
+                    <mesh filename="package://edo_description/meshes/visual/base_spacer.stl"/>
                 </geometry>
                 <material name="Grey"/>
@@ -73,5 +73,5 @@
                 <origin xyz="0 0 0" rpy="0 0 0"/>
                 <geometry>
-                    <mesh filename="package://edo_description/meshes/base_spacer.stl"/>
+                    <mesh filename="package://edo_description/meshes/collision/base_spacer.stl"/>
                 </geometry>
                 <material name="Grey"/>
@@ -103,12 +103,12 @@
                 <origin xyz="0 0 0" rpy="0 0 0"/>
                 <geometry>
-                    <mesh filename="package://edo_description/meshes/link_1.stl"/>
-                </geometry>
-                <material name="Orange"/>
-            </visual>
-            <collision>
-                <origin xyz="0 0 0" rpy="0 0 0"/>
-                <geometry>
-                    <mesh filename="package://edo_description/meshes/link_1.stl"/>
+                    <mesh filename="package://edo_description/meshes/visual/link_1.stl"/>
+                </geometry>
+                <material name="Orange"/>
+            </visual>
+            <collision>
+                <origin xyz="0 0 0" rpy="0 0 0"/>
+                <geometry>
+                    <mesh filename="package://edo_description/meshes/collision/link_1.stl"/>
                 </geometry>
                 <material name="Orange"/>
@@ -139,12 +139,12 @@
                 <origin xyz="0 0 0" rpy="0 0 0"/>
                 <geometry>
-                    <mesh filename="package://edo_description/meshes/link_2.stl"/>
-                </geometry>
-                <material name="Orange"/>
-            </visual>
-            <collision>
-                <origin xyz="0 0 0" rpy="0 0 0"/>
-                <geometry>
-                    <mesh filename="package://edo_description/meshes/link_2.stl"/>
+                    <mesh filename="package://edo_description/meshes/visual/link_2.stl"/>
+                </geometry>
+                <material name="Orange"/>
+            </visual>
+            <collision>
+                <origin xyz="0 0 0" rpy="0 0 0"/>
+                <geometry>
+                    <mesh filename="package://edo_description/meshes/collision/link_2.stl"/>
                 </geometry>
                 <material name="Orange"/>
@@ -175,12 +175,12 @@
                 <origin xyz="0 0 0" rpy="0 0 0"/>
                 <geometry>
-                    <mesh filename="package://edo_description/meshes/link_3.stl"/>
-                </geometry>
-                <material name="Orange"/>
-            </visual>
-            <collision>
-                <origin xyz="0 0 0" rpy="0 0 0"/>
-                <geometry>
-                    <mesh filename="package://edo_description/meshes/link_3.stl"/>
+                    <mesh filename="package://edo_description/meshes/visual/link_3.stl"/>
+                </geometry>
+                <material name="Orange"/>
+            </visual>
+            <collision>
+                <origin xyz="0 0 0" rpy="0 0 0"/>
+                <geometry>
+                    <mesh filename="package://edo_description/meshes/collision/link_3.stl"/>
                 </geometry>
                 <material name="Orange"/>
@@ -211,12 +211,12 @@
                 <origin xyz="0 0 0" rpy="0 0 0"/>
                 <geometry>
-                    <mesh filename="package://edo_description/meshes/link_4.stl"/>
-                </geometry>
-                <material name="Orange"/>
-            </visual>
-            <collision>
-                <origin xyz="0 0 0" rpy="0 0 0"/>
-                <geometry>
-                    <mesh filename="package://edo_description/meshes/link_4.stl"/>
+                    <mesh filename="package://edo_description/meshes/visual/link_4.stl"/>
+                </geometry>
+                <material name="Orange"/>
+            </visual>
+            <collision>
+                <origin xyz="0 0 0" rpy="0 0 0"/>
+                <geometry>
+                    <mesh filename="package://edo_description/meshes/collision/link_4.stl"/>
                 </geometry>
                 <material name="Orange"/>
@@ -247,12 +247,12 @@
                 <origin xyz="0 0 0" rpy="0 0 0"/>
                 <geometry>
-                    <mesh filename="package://edo_description/meshes/link_5.stl"/>
-                </geometry>
-                <material name="Orange"/>
-            </visual>
-            <collision>
-                <origin xyz="0 0 0" rpy="0 0 0"/>
-                <geometry>
-                    <mesh filename="package://edo_description/meshes/link_5.stl"/>
+                    <mesh filename="package://edo_description/meshes/visual/link_5.stl"/>
+                </geometry>
+                <material name="Orange"/>
+            </visual>
+            <collision>
+                <origin xyz="0 0 0" rpy="0 0 0"/>
+                <geometry>
+                    <mesh filename="package://edo_description/meshes/collision/link_5.stl"/>
                 </geometry>
                 <material name="Orange"/>
@@ -286,12 +286,12 @@
                 <origin xyz="0 0 0" rpy="0 0 0"/>
                 <geometry>
-                    <mesh filename="package://edo_description/meshes/link_6.stl"/>
-                </geometry>
-                <material name="Orange"/>
-            </visual>
-            <collision>
-                <origin xyz="0 0 0" rpy="0 0 0"/>
-                <geometry>
-                    <mesh filename="package://edo_description/meshes/link_6.stl"/>
+                    <mesh filename="package://edo_description/meshes/visual/link_6.stl"/>
+                </geometry>
+                <material name="Orange"/>
+            </visual>
+            <collision>
+                <origin xyz="0 0 0" rpy="0 0 0"/>
+                <geometry>
+                    <mesh filename="package://edo_description/meshes/collision/link_6.stl"/>
                 </geometry>
                 <material name="Orange"/>

Commit message: Fix wobbling of robot

File: urdf/edo.xacro (robot description, xacro)
@@ -83,6 +83,6 @@
             <parent link="${robot_name}_link_1"/>
             <child link="${robot_name}_link_2"/>
-            <origin xyz="0 0 0" rpy="0 0 0"/>
-            <axis xyz="0 1 0"/>
+            <origin xyz="0 0 0" rpy="${PI /2} 0 0"/>
+            <axis xyz="0 0 -1"/>
             <limit lower="${-113 * PI / 180}" upper="${113 * PI / 180}"
                    effort="${max_effort}" velocity="${max_velocity}" />
@@ -102,5 +102,5 @@
             </inertial>
             <visual>
-                <origin xyz="0 0 0.2105" rpy="0 0 0"/>
+                <origin xyz="0 0.2105 0" rpy="${PI /2} ${PI} ${PI}"/>
                 <geometry>
                     <mesh filename="package://edo_description/meshes/visual/link_2.dae"/>
@@ -108,5 +108,5 @@
             </visual>
             <collision>
-                <origin xyz="0 0 0.2105" rpy="0 0 0"/>
+                <origin xyz="0 0.2105 0" rpy="${PI /2} ${PI} ${PI}"/>
                 <geometry>
                     <mesh filename="package://edo_description/meshes/collision/link_2.dae"/>
@@ -118,6 +118,6 @@
             <parent link="${robot_name}_link_2"/>
             <child link="${robot_name}_link_3"/>
-            <origin xyz="0 0 0.2105" rpy="0 0 0"/>
-            <axis xyz="0 1 0"/>
+            <origin xyz="0 0.2105 0" rpy="0 ${PI} ${PI}"/>
+            <axis xyz="0 0 1"/>
             <limit lower="${-113 * PI / 180}" upper="${113 * PI / 180}"
                    effort="${max_effort}" velocity="${max_velocity}" />
@@ -137,5 +137,5 @@
             </inertial>
             <visual>
-                <origin xyz="0 0 0" rpy="0 0 0"/>
+                <origin xyz="0 0 0" rpy="${PI /2} 0 0"/>
                 <geometry>
                     <mesh filename="package://edo_description/meshes/visual/link_3.dae"/>
@@ -143,5 +143,5 @@
             </visual>
             <collision>
-                <origin xyz="0 0 0" rpy="0 0 0"/>
+                <origin xyz="0 0 0" rpy="${PI /2} 0 0"/>
                 <geometry>
                     <mesh filename="package://edo_description/meshes/collision/link_3.dae"/>
@@ -153,5 +153,5 @@
             <parent link="${robot_name}_link_3"/>
             <child link="${robot_name}_link_4"/>
-            <origin xyz="0 0 0.268" rpy="0 0 0"/>
+            <origin xyz="0 -0.268 0" rpy="${PI / 2} 0 0"/>
             <axis xyz="0 0 1"/>
             <limit lower="${-180 * PI / 180}" upper="${180 * PI / 180}"

Commit message: Set real world robot joint limits.
The technical sheet has listed bigger joint limits than the robot/eORL can reach.

File: urdf/edo.xacro (robot description, xacro)
@@ -50,5 +50,6 @@
             <origin xyz="0 0 ${0.135 + 0.202}" rpy="0 0 0"/>
             <axis xyz="0 0 1"/>
-            <limit lower="${-180 * PI / 180}" upper="${180 * PI / 180}"
+            <!-- Joint limits of the real robot determined by jogging. TechSheet is wrong -->
+            <limit lower="${-178 * PI / 180}" upper="${178 * PI / 180}"
                    effort="${max_effort}" velocity="${max_velocity}" />
             <dynamics damping="${joint_damping}"/>
@@ -85,5 +86,6 @@
             <origin xyz="0 0 0" rpy="${PI /2} 0 0"/>
             <axis xyz="0 0 -1"/>
-            <limit lower="${-113 * PI / 180}" upper="${113 * PI / 180}"
+            <!-- Joint limits of the real robot determined by jogging. TechSheet is wrong -->
+            <limit lower="${-98 * PI / 180}" upper="${98 * PI / 180}"
                    effort="${max_effort}" velocity="${max_velocity}" />
             <dynamics damping="${joint_damping}"/>
@@ -120,5 +122,6 @@
             <origin xyz="0 0.2105 0" rpy="0 ${PI} ${PI}"/>
             <axis xyz="0 0 1"/>
-            <limit lower="${-113 * PI / 180}" upper="${113 * PI / 180}"
+            <!-- Joint limits of the real robot determined by jogging. TechSheet is wrong -->
+            <limit lower="${-98 * PI / 180}" upper="${98 * PI / 180}"
                    effort="${max_effort}" velocity="${max_velocity}" />
             <dynamics damping="${joint_damping}"/>
@@ -155,5 +158,6 @@
             <origin xyz="0 -0.268 0" rpy="${PI / 2} 0 0"/>
             <axis xyz="0 0 1"/>
-            <limit lower="${-180 * PI / 180}" upper="${180 * PI / 180}"
+            <!-- Joint limits of the real robot determined by jogging. TechSheet is wrong -->
+            <limit lower="${-178 * PI / 180}" upper="${178 * PI / 180}"
                    effort="${max_effort}" velocity="${max_velocity}" />
             <dynamics damping="${joint_damping}"/>
@@ -190,5 +194,6 @@
             <origin xyz="0 0 0" rpy="0 0 0"/>
             <axis xyz="0 1 0"/>
-            <limit lower="${-104 * PI / 180}" upper="${104 * PI / 180}"
+            <!-- Joint limits of the real robot determined by jogging. TechSheet is wrong -->
+            <limit lower="${-103 * PI / 180}" upper="${103 * PI / 180}"
                    effort="${max_effort}" velocity="${max_velocity}" />
             <dynamics damping="${joint_damping}"/>
