Commit message: New colorized simulation model

File: urdf/edo.gazebo.xacro (robot description, xacro)
@@ -9,6 +9,5 @@
         </gazebo>
         <!-- Link0 -->
-        <gazebo reference="${robot_name}_link_0">
-            <material>Gazebo/Grey</material>
+        <gazebo reference="${robot_name}_base_link">
             <mu1>0.2</mu1>
             <mu2>0.2</mu2>
@@ -16,5 +15,4 @@
         <!-- Link1 -->
         <gazebo reference="${robot_name}_link_1">
-            <material>Gazebo/Orange</material>
             <mu1>0.2</mu1>
             <mu2>0.2</mu2>
@@ -22,5 +20,4 @@
         <!-- Link2 -->
         <gazebo reference="${robot_name}_link_2">
-            <material>Gazebo/Orange</material>
             <mu1>0.2</mu1>
             <mu2>0.2</mu2>
@@ -28,5 +25,4 @@
         <!-- Link3 -->
         <gazebo reference="${robot_name}_link_3">
-            <material>Gazebo/Orange</material>
             <mu1>0.2</mu1>
             <mu2>0.2</mu2>
@@ -34,5 +30,4 @@
         <!-- Link4 -->
         <gazebo reference="${robot_name}_link_4">
-            <material>Gazebo/Orange</material>
             <mu1>0.2</mu1>
             <mu2>0.2</mu2>
@@ -40,5 +35,4 @@
         <!-- Link5 -->
         <gazebo reference="${robot_name}_link_5">
-            <material>Gazebo/Orange</material>
             <mu1>0.2</mu1>
             <mu2>0.2</mu2>
@@ -46,5 +40,4 @@
         <!-- Link6 -->
         <gazebo reference="${robot_name}_link_6">
-            <material>Gazebo/Orange</material>
             <mu1>0.2</mu1>
             <mu2>0.2</mu2>

File: urdf/edo.xacro (robot description, xacro)
@@ -31,47 +31,13 @@
             </inertial>
             <visual>
-                <origin xyz="0 0 0" rpy="0 0 0"/>
-                <geometry>
-                    <mesh filename="package://edo_description/meshes/visual/base_link.stl"/>
-                </geometry>
-                <material name="Grey"/>
-            </visual>
-            <collision>
-                <origin xyz="0 0 0" rpy="0 0 0"/>
-                <geometry>
-                    <mesh filename="package://edo_description/meshes/collision/base_link.stl"/>
-                </geometry>
-                <material name="Grey"/>
-            </collision>
-        </link>
-        <!-- joint between base_link and base_spacer -->
-        <joint name="${robot_name}_joint_spacer" type="fixed">
-            <parent link="${robot_name}_base_link"/>
-            <child link="${robot_name}_base_spacer_link"/>
-            <origin xyz="0 0 0.135" rpy="0 0 0"/>
-        </joint>
-        <link name="${robot_name}_base_spacer_link">
-            <inertial>
-                <origin xyz="0 0 0.005" rpy="0 0 0"/>
-                <mass value="0.01"/>
-                <inertia
-                        ixx="0.0123841200738068"
-                        ixy="-0.000187984913202787"
-                        ixz="-1.32683892634308E-06"
-                        iyy="7.0169034503364E-05"
-                        iyz="-9.17416945099319E-05"
-                        izz="0.0123862261905614" />
-            </inertial>
-            <visual>
-                <origin xyz="0 0 0" rpy="0 0 0"/>
-                <geometry>
-                    <mesh filename="package://edo_description/meshes/visual/base_spacer.stl"/>
-                </geometry>
-                <material name="Grey"/>
-            </visual>
-            <collision>
-                <origin xyz="0 0 0" rpy="0 0 0"/>
-                <geometry>
-                    <mesh filename="package://edo_description/meshes/collision/base_spacer.stl"/>
+                <origin xyz="0 0 0.135" rpy="0 0 0"/>
+                <geometry>
+                    <mesh filename="package://edo_description/meshes/visual/link_0.dae"/>
+                </geometry>
+            </visual>
+            <collision>
+                <origin xyz="0 0 0.135" rpy="0 0 0"/>
+                <geometry>
+                    <mesh filename="package://edo_description/meshes/collision/link_0.dae"/>
                 </geometry>
                 <material name="Grey"/>
@@ -103,12 +69,11 @@
                 <origin xyz="0 0 0" rpy="0 0 0"/>
                 <geometry>
-                    <mesh filename="package://edo_description/meshes/visual/link_1.stl"/>
-                </geometry>
-                <material name="Orange"/>
-            </visual>
-            <collision>
-                <origin xyz="0 0 0" rpy="0 0 0"/>
-                <geometry>
-                    <mesh filename="package://edo_description/meshes/collision/link_1.stl"/>
+                    <mesh filename="package://edo_description/meshes/visual/link_1.dae"/>
+                </geometry>
+            </visual>
+            <collision>
+                <origin xyz="0 0 0" rpy="0 0 0"/>
+                <geometry>
+                    <mesh filename="package://edo_description/meshes/collision/link_1.dae"/>
                 </geometry>
                 <material name="Orange"/>
@@ -118,6 +83,6 @@
             <parent link="${robot_name}_link_1"/>
             <child link="${robot_name}_link_2"/>
-            <origin xyz="0 0 0" rpy="${PI /2} 0 0"/>
-            <axis xyz="0 0 -1"/>
+            <origin xyz="0 0 0" rpy="0 0 0"/>
+            <axis xyz="0 1 0"/>
             <limit lower="${-113 * PI / 180}" upper="${113 * PI / 180}"
                    effort="${max_effort}" velocity="${max_velocity}" />
@@ -137,14 +102,13 @@
             </inertial>
             <visual>
-                <origin xyz="0 0 0" rpy="0 0 0"/>
-                <geometry>
-                    <mesh filename="package://edo_description/meshes/visual/link_2.stl"/>
-                </geometry>
-                <material name="Orange"/>
-            </visual>
-            <collision>
-                <origin xyz="0 0 0" rpy="0 0 0"/>
-                <geometry>
-                    <mesh filename="package://edo_description/meshes/collision/link_2.stl"/>
+                <origin xyz="0 0 0.2105" rpy="0 0 0"/>
+                <geometry>
+                    <mesh filename="package://edo_description/meshes/visual/link_2.dae"/>
+                </geometry>
+            </visual>
+            <collision>
+                <origin xyz="0 0 0.2105" rpy="0 0 0"/>
+                <geometry>
+                    <mesh filename="package://edo_description/meshes/collision/link_2.dae"/>
                 </geometry>
                 <material name="Orange"/>
@@ -154,6 +118,6 @@
             <parent link="${robot_name}_link_2"/>
             <child link="${robot_name}_link_3"/>
-            <origin xyz="0 0.2105 0" rpy="0 ${PI} ${PI}"/>
-            <axis xyz="0 0 1"/>
+            <origin xyz="0 0 0.2105" rpy="0 0 0"/>
+            <axis xyz="0 1 0"/>
             <limit lower="${-113 * PI / 180}" upper="${113 * PI / 180}"
                    effort="${max_effort}" velocity="${max_velocity}" />
@@ -175,12 +139,11 @@
                 <origin xyz="0 0 0" rpy="0 0 0"/>
                 <geometry>
-                    <mesh filename="package://edo_description/meshes/visual/link_3.stl"/>
-                </geometry>
-                <material name="Orange"/>
-            </visual>
-            <collision>
-                <origin xyz="0 0 0" rpy="0 0 0"/>
-                <geometry>
-                    <mesh filename="package://edo_description/meshes/collision/link_3.stl"/>
+                    <mesh filename="package://edo_description/meshes/visual/link_3.dae"/>
+                </geometry>
+            </visual>
+            <collision>
+                <origin xyz="0 0 0" rpy="0 0 0"/>
+                <geometry>
+                    <mesh filename="package://edo_description/meshes/collision/link_3.dae"/>
                 </geometry>
                 <material name="Orange"/>
@@ -190,5 +153,5 @@
             <parent link="${robot_name}_link_3"/>
             <child link="${robot_name}_link_4"/>
-            <origin xyz="0 -0.268 0" rpy="${PI / 2} 0 0"/>
+            <origin xyz="0 0 0.268" rpy="0 0 0"/>
             <axis xyz="0 0 1"/>
             <limit lower="${-180 * PI / 180}" upper="${180 * PI / 180}"
@@ -211,12 +174,11 @@
                 <origin xyz="0 0 0" rpy="0 0 0"/>
                 <geometry>
-                    <mesh filename="package://edo_description/meshes/visual/link_4.stl"/>
-                </geometry>
-                <material name="Orange"/>
-            </visual>
-            <collision>
-                <origin xyz="0 0 0" rpy="0 0 0"/>
-                <geometry>
-                    <mesh filename="package://edo_description/meshes/collision/link_4.stl"/>
+                    <mesh filename="package://edo_description/meshes/visual/link_4.dae"/>
+                </geometry>
+            </visual>
+            <collision>
+                <origin xyz="0 0 0" rpy="0 0 0"/>
+                <geometry>
+                    <mesh filename="package://edo_description/meshes/collision/link_4.dae"/>
                 </geometry>
                 <material name="Orange"/>
@@ -247,12 +209,11 @@
                 <origin xyz="0 0 0" rpy="0 0 0"/>
                 <geometry>
-                    <mesh filename="package://edo_description/meshes/visual/link_5.stl"/>
-                </geometry>
-                <material name="Orange"/>
-            </visual>
-            <collision>
-                <origin xyz="0 0 0" rpy="0 0 0"/>
-                <geometry>
-                    <mesh filename="package://edo_description/meshes/collision/link_5.stl"/>
+                    <mesh filename="package://edo_description/meshes/visual/link_5.dae"/>
+                </geometry>
+            </visual>
+            <collision>
+                <origin xyz="0 0 0" rpy="0 0 0"/>
+                <geometry>
+                    <mesh filename="package://edo_description/meshes/collision/link_5.dae"/>
                 </geometry>
                 <material name="Orange"/>
@@ -286,12 +247,11 @@
                 <origin xyz="0 0 0" rpy="0 0 0"/>
                 <geometry>
-                    <mesh filename="package://edo_description/meshes/visual/link_6.stl"/>
-                </geometry>
-                <material name="Orange"/>
-            </visual>
-            <collision>
-                <origin xyz="0 0 0" rpy="0 0 0"/>
-                <geometry>
-                    <mesh filename="package://edo_description/meshes/collision/link_6.stl"/>
+                    <mesh filename="package://edo_description/meshes/visual/link_6.dae"/>
+                </geometry>
+            </visual>
+            <collision>
+                <origin xyz="0 0 0" rpy="0 0 0"/>
+                <geometry>
+                    <mesh filename="package://edo_description/meshes/collision/link_6.dae"/>
                 </geometry>
                 <material name="Orange"/>
