Commit message: Correctly handle robot name to allow adding multiple instances

File: urdf/edo.gazebo.xacro (robot description, xacro)
@@ -1,5 +1,5 @@
 <?xml version="1.0"?>
 <robot xmlns:xacro="http://www.ros.org/wiki/xacro">
-    <xacro:macro name="edo_gazebo" params="robot_name">
+    <xacro:macro name="edo_gazebo" params="robot_name robot_prefix">
         <!-- Load Gazebo lib and set the robot namespace -->
         <gazebo>
@@ -9,35 +9,35 @@
         </gazebo>
         <!-- Link0 -->
-        <gazebo reference="${robot_name}_base_link">
+        <gazebo reference="${robot_prefix}_base_link">
             <mu1>0.2</mu1>
             <mu2>0.2</mu2>
         </gazebo>
         <!-- Link1 -->
-        <gazebo reference="${robot_name}_link_1">
+        <gazebo reference="${robot_prefix}_link_1">
             <mu1>0.2</mu1>
             <mu2>0.2</mu2>
         </gazebo>
         <!-- Link2 -->
-        <gazebo reference="${robot_name}_link_2">
+        <gazebo reference="${robot_prefix}_link_2">
             <mu1>0.2</mu1>
             <mu2>0.2</mu2>
         </gazebo>
         <!-- Link3 -->
-        <gazebo reference="${robot_name}_link_3">
+        <gazebo reference="${robot_prefix}_link_3">
             <mu1>0.2</mu1>
             <mu2>0.2</mu2>
         </gazebo>
         <!-- Link4 -->
-        <gazebo reference="${robot_name}_link_4">
+        <gazebo reference="${robot_prefix}_link_4">
             <mu1>0.2</mu1>
             <mu2>0.2</mu2>
         </gazebo>
         <!-- Link5 -->
-        <gazebo reference="${robot_name}_link_5">
+        <gazebo reference="${robot_prefix}_link_5">
             <mu1>0.2</mu1>
             <mu2>0.2</mu2>
         </gazebo>
         <!-- Link6 -->
-        <gazebo reference="${robot_name}_link_6">
+        <gazebo reference="${robot_prefix}_link_6">
             <mu1>0.2</mu1>
             <mu2>0.2</mu2>

File: urdf/edo.transmission.xacro (robot description, xacro)
@@ -2,66 +2,66 @@
 <robot xmlns:xacro="http://www.ros.org/wiki/xacro">
     <xacro:macro name="edo_transmission" params="hardware_interface">
-        <transmission name="${robot_name}_tran_1">
+        <transmission name="${robot_prefix}_tran_1">
             <robotNamespace>/${robot_name}</robotNamespace>
             <type>transmission_interface/SimpleTransmission</type>
-            <joint name="${robot_name}_joint_1">
+            <joint name="${robot_prefix}_joint_1">
                 <hardwareInterface>${hardware_interface}</hardwareInterface>
             </joint>
-            <actuator name="${robot_name}_motor_1">
+            <actuator name="${robot_prefix}_motor_1">
                 <hardwareInterface>${hardware_interface}</hardwareInterface>
                 <mechanicalReduction>1</mechanicalReduction>
             </actuator>
         </transmission>
-        <transmission name="${robot_name}_tran_2">
+        <transmission name="${robot_prefix}_tran_2">
             <robotNamespace>/${robot_name}</robotNamespace>
             <type>transmission_interface/SimpleTransmission</type>
-            <joint name="${robot_name}_joint_2">
+            <joint name="${robot_prefix}_joint_2">
                 <hardwareInterface>${hardware_interface}</hardwareInterface>
             </joint>
-            <actuator name="${robot_name}_motor_2">
+            <actuator name="${robot_prefix}_motor_2">
                 <hardwareInterface>${hardware_interface}</hardwareInterface>
                 <mechanicalReduction>1</mechanicalReduction>
             </actuator>
         </transmission>
-        <transmission name="${robot_name}_tran_3">
+        <transmission name="${robot_prefix}_tran_3">
             <robotNamespace>/${robot_name}</robotNamespace>
             <type>transmission_interface/SimpleTransmission</type>
-            <joint name="${robot_name}_joint_3">
+            <joint name="${robot_prefix}_joint_3">
                 <hardwareInterface>${hardware_interface}</hardwareInterface>
             </joint>
-            <actuator name="${robot_name}_motor_3">
+            <actuator name="${robot_prefix}_motor_3">
                 <hardwareInterface>${hardware_interface}</hardwareInterface>
                 <mechanicalReduction>1</mechanicalReduction>
             </actuator>
         </transmission>
-        <transmission name="${robot_name}_tran_4">
+        <transmission name="${robot_prefix}_tran_4">
             <robotNamespace>/${robot_name}</robotNamespace>
             <type>transmission_interface/SimpleTransmission</type>
-            <joint name="${robot_name}_joint_4">
+            <joint name="${robot_prefix}_joint_4">
                 <hardwareInterface>${hardware_interface}</hardwareInterface>
             </joint>
-            <actuator name="${robot_name}_motor_4">
+            <actuator name="${robot_prefix}_motor_4">
                 <hardwareInterface>${hardware_interface}</hardwareInterface>
                 <mechanicalReduction>1</mechanicalReduction>
             </actuator>
         </transmission>
-        <transmission name="${robot_name}_tran_5">
+        <transmission name="${robot_prefix}_tran_5">
             <robotNamespace>/${robot_name}</robotNamespace>
             <type>transmission_interface/SimpleTransmission</type>
-            <joint name="${robot_name}_joint_5">
+            <joint name="${robot_prefix}_joint_5">
                 <hardwareInterface>${hardware_interface}</hardwareInterface>
             </joint>
-            <actuator name="${robot_name}_motor_5">
+            <actuator name="${robot_prefix}_motor_5">
                 <hardwareInterface>${hardware_interface}</hardwareInterface>
                 <mechanicalReduction>1</mechanicalReduction>
             </actuator>
         </transmission>
-        <transmission name="${robot_name}_tran_6">
+        <transmission name="${robot_prefix}_tran_6">
             <robotNamespace>/${robot_name}</robotNamespace>
             <type>transmission_interface/SimpleTransmission</type>
-            <joint name="${robot_name}_joint_6">
+            <joint name="${robot_prefix}_joint_6">
                 <hardwareInterface>${hardware_interface}</hardwareInterface>
             </joint>
-            <actuator name="${robot_name}_motor_6">
+            <actuator name="${robot_prefix}_motor_6">
                 <hardwareInterface>${hardware_interface}</hardwareInterface>
                 <mechanicalReduction>1</mechanicalReduction>

File: urdf/edo.xacro (robot description, xacro)
@@ -11,4 +11,5 @@
     <xacro:property name="max_effort" value="300"/>
     <xacro:property name="max_velocity" value="1.5"/>
+    <xacro:property name="robot_prefix" value="edo"/>
     <xacro:macro name="edo" params="parent hardware_interface robot_name *origin">
         <!--joint between {parent} and base_link-->
@@ -16,7 +17,7 @@
             <xacro:insert_block name="origin"/>
             <parent link="${parent}"/>
-            <child link="${robot_name}_base_link"/>
-        </joint>
-        <link name="${robot_name}_base_link">
+            <child link="${robot_prefix}_base_link"/>
+        </joint>
+        <link name="${robot_prefix}_base_link">
             <inertial>
                 <origin xyz="0.057188 0.005983 0.05" rpy="0 0 0"/>
@@ -45,7 +46,7 @@
         </link>
         <!-- joint between base_link and link_1 -->
-        <joint name="${robot_name}_joint_1" type="revolute">
-            <parent link="${robot_name}_base_link"/>
-            <child link="${robot_name}_link_1"/>
+        <joint name="${robot_prefix}_joint_1" type="revolute">
+            <parent link="${robot_prefix}_base_link"/>
+            <child link="${robot_prefix}_link_1"/>
             <origin xyz="0 0 ${0.135 + 0.202}" rpy="0 0 0"/>
             <axis xyz="0 0 1"/>
@@ -55,5 +56,5 @@
             <dynamics damping="${joint_damping}"/>
         </joint>
-        <link name="${robot_name}_link_1">
+        <link name="${robot_prefix}_link_1">
             <inertial>
                 <origin xyz="-0.037464 0.047260 0" rpy="0 0 0"/>
@@ -81,7 +82,7 @@
             </collision>
         </link>
-        <joint name="${robot_name}_joint_2" type="revolute">
-            <parent link="${robot_name}_link_1"/>
-            <child link="${robot_name}_link_2"/>
+        <joint name="${robot_prefix}_joint_2" type="revolute">
+            <parent link="${robot_prefix}_link_1"/>
+            <child link="${robot_prefix}_link_2"/>
             <origin xyz="0 0 0" rpy="${PI /2} 0 0"/>
             <axis xyz="0 0 -1"/>
@@ -91,5 +92,5 @@
             <dynamics damping="${joint_damping}"/>
         </joint>
-        <link name="${robot_name}_link_2">
+        <link name="${robot_prefix}_link_2">
             <inertial>
                 <origin xyz="-0.016423 0.031803 -0.045948" rpy="0 0 0"/>
@@ -117,7 +118,7 @@
             </collision>
         </link>
-        <joint name="${robot_name}_joint_3" type="revolute">
-            <parent link="${robot_name}_link_2"/>
-            <child link="${robot_name}_link_3"/>
+        <joint name="${robot_prefix}_joint_3" type="revolute">
+            <parent link="${robot_prefix}_link_2"/>
+            <child link="${robot_prefix}_link_3"/>
             <origin xyz="0 0.2105 0" rpy="0 ${PI} ${PI}"/>
             <axis xyz="0 0 1"/>
@@ -127,5 +128,5 @@
             <dynamics damping="${joint_damping}"/>
         </joint>
-        <link name="${robot_name}_link_3">
+        <link name="${robot_prefix}_link_3">
             <inertial>
                 <origin xyz="-0.031475 0.013100 0.000326" rpy="0 0 0"/>
@@ -153,7 +154,7 @@
             </collision>
         </link>
-        <joint name="${robot_name}_joint_4" type="revolute">
-            <parent link="${robot_name}_link_3"/>
-            <child link="${robot_name}_link_4"/>
+        <joint name="${robot_prefix}_joint_4" type="revolute">
+            <parent link="${robot_prefix}_link_3"/>
+            <child link="${robot_prefix}_link_4"/>
             <origin xyz="0 -0.268 0" rpy="${PI / 2} 0 0"/>
             <axis xyz="0 0 1"/>
@@ -163,5 +164,5 @@
             <dynamics damping="${joint_damping}"/>
         </joint>
-        <link name="${robot_name}_link_4">
+        <link name="${robot_prefix}_link_4">
             <inertial>
                 <origin xyz="0.033909 0.000544 -0.013765" rpy="0 0 0"/>
@@ -189,7 +190,7 @@
             </collision>
         </link>
-        <joint name="${robot_name}_joint_5" type="revolute">
-            <parent link="${robot_name}_link_4"/>
-            <child link="${robot_name}_link_5"/>
+        <joint name="${robot_prefix}_joint_5" type="revolute">
+            <parent link="${robot_prefix}_link_4"/>
+            <child link="${robot_prefix}_link_5"/>
             <origin xyz="0 0 0" rpy="0 0 0"/>
             <axis xyz="0 1 0"/>
@@ -199,5 +200,5 @@
             <dynamics damping="${joint_damping}"/>
         </joint>
-        <link name="${robot_name}_link_5">
+        <link name="${robot_prefix}_link_5">
             <inertial>
                 <origin xyz="0.029485 -0.000458 0.026739" rpy="0 0 0"/>
@@ -225,7 +226,7 @@
             </collision>
         </link>
-        <joint name="${robot_name}_joint_6" type="revolute">
-            <parent link="${robot_name}_link_5"/>
-            <child link="${robot_name}_link_6"/>
+        <joint name="${robot_prefix}_joint_6" type="revolute">
+            <parent link="${robot_prefix}_link_5"/>
+            <child link="${robot_prefix}_link_6"/>
             <origin xyz="0 0 0.1745" rpy="0 0 0"/>
             <axis xyz="0 0 1"/>
@@ -237,5 +238,5 @@
             <dynamics damping="${joint_damping}"/>
         </joint>
-        <link name="${robot_name}_link_6">
+        <link name="${robot_prefix}_link_6">
             <inertial>
                 <origin xyz="0.000007 -0.009327 0.000006" rpy="0 0 0"/>
@@ -263,13 +264,13 @@
             </collision>
         </link>
-        <joint name="${robot_name}_joint_ee" type="fixed">
-            <parent link="${robot_name}_link_6"/>
-            <child link="${robot_name}_link_ee"/>
+        <joint name="${robot_prefix}_joint_ee" type="fixed">
+            <parent link="${robot_prefix}_link_6"/>
+            <child link="${robot_prefix}_link_ee"/>
             <origin xyz="0 0 0" rpy="0 0 0"/>
         </joint>
-        <link name="${robot_name}_link_ee">
+        <link name="${robot_prefix}_link_ee">
         </link>
         <!--Extensions -->
-        <xacro:edo_gazebo robot_name="${robot_name}" />
+        <xacro:edo_gazebo robot_name="${robot_name}" robot_prefix="${robot_prefix}" />
         <xacro:edo_transmission hardware_interface="${hardware_interface}"/>
     </xacro:macro>
